Commit message: Update ur5.urdf.xacro

File: packages/ur5/ros2srrc_ur5_gazebo/urdf/ur5.urdf.xacro (robot description, xacro)
@@ -80,5 +80,5 @@
       <origin xyz="0 0 0" rpy=" 0 0 0"/>
       <geometry>
-        <box size = "0.2 0.2 0.5"/>
+        <box size = "0.2 0.2 1.0"/>
       </geometry>
     </collision>
@@ -86,5 +86,5 @@
       <origin xyz="0 0 0" rpy=" 0 0 0"/>
       <geometry>
-        <box size = "0.2 0.2 0.5"/>
+        <box size = "0.2 0.2 1.0"/>
       </geometry>
     </visual>
@@ -94,5 +94,5 @@
     <parent link= "world" />
     <child link = "robot_stand" />
-    <origin xyz="0.0 0.0 0.25" rpy="0.0 0.0 0.0" />
+    <origin xyz="0.0 0.0 0.5" rpy="0.0 0.0 0.0" />
   </joint>
   <!-- Robot Stand: Robot+Stand JOINT -->
@@ -100,5 +100,5 @@
     <parent link= "robot_stand" />
     <child link = "base_link" />
-    <origin xyz="0.0 0.0 0.255" rpy="0.0 0.0 0.0" />
+    <origin xyz="0.0 0.0 0.501" rpy="0.0 0.0 0.0" />
   </joint>
   <!-- ros2srrc_HMI CAMERA -->
