Commit message: Change the height

File: packages/ur5/ros2srrc_ur5_gazebo/urdf/ur5_robotiq_hande.urdf.xacro (robot description, xacro)
@@ -102,5 +102,5 @@
     <parent link= "world" />
     <child link = "robot_stand" />
-    <origin xyz="0.0 0.0 0.25" rpy="0.0 0.0 0.0" />
+    <origin xyz="0.0 0.0 0.5" rpy="0.0 0.0 0.0" />
   </joint>
   <!-- Robot Stand: Robot+Stand JOINT -->
@@ -108,5 +108,5 @@
     <parent link= "robot_stand" />
     <child link = "base_link" />
-    <origin xyz="0.0 0.0 0.255" rpy="0.0 0.0 0.0" />
+    <origin xyz="0.0 0.0 0.501" rpy="0.0 0.0 0.0" />
   </joint>
   <!-- ros2srrc_HMI CAMERA -->

Commit message: Add more height

File: packages/ur5/ros2srrc_ur5_gazebo/urdf/ur5_robotiq_hande.urdf.xacro (robot description, xacro)
@@ -88,5 +88,5 @@
       <origin xyz="0 0 0" rpy=" 0 0 0"/>
       <geometry>
-        <box size = "0.2 0.2 0.5"/>
+        <box size = "0.2 0.2 1.0"/>
       </geometry>
     </collision>
@@ -94,5 +94,5 @@
       <origin xyz="0 0 0" rpy=" 0 0 0"/>
       <geometry>
-        <box size = "0.2 0.2 0.5"/>
+        <box size = "0.2 0.2 1.0"/>
       </geometry>
     </visual>
